File: CW312T-EFR32MG21-SOCKET.kicad_sch (KiCad schematic)
At the start: 18 parts, among them J1 1x3 straight header pins, P1 PCIEx4 EDGE CONNECTOR, U1 EFR32MG21A020F1024IM32-BR

Commit message: first draft - ready for review
Parts:
- added PCB1: CE Symbol, Silkscrren_Symbols:CE-Logo_8.5x6mm_SilkScreen, symbol Silkscreen_Symbols:CE_Free
- added PCB2: Pb_Free Symbol, Silkscrren_Symbols:Pb_Free_8.0x8.0mm_SilkScreen, symbol Silkscreen_Symbols:Pb_Free
- added PCB3: UKCA symbol, Silkscrren_Symbols:UKCA-Logo_8x8mm_SilkScreen, symbol Silkscreen_Symbols:UKCA
- added PCB4: WEEE SYMBOL, Silkscrren_Symbols:WEEE-Logo_5.6x8mm_SilkScreen, symbol Silkscreen_Symbols:WEEE

Commit message: updated schematic, pcb and production files - Ready for review
Connections:
- net +3V3: now also P1.A26 (JTAG_VREF)
- no-connect marks 47 -> 46
Other:
- note added: "Need to confirm the footprint of the socket - the one included in production files does not have a model but an equivalent socket on digikey did so i used that downloaded model"
- note added: "cw308 schematic includes note bubbles stating 'morespace' i left those out but can include if preferred"
- note removed: "Need to confirm the footprint of the socket - the one included in production files does not have a model but an equivalent socket on digikey did"
Changed lines of the file:
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@@
+	)
+	(junction
+		(at 39.37 62.23)
+		(diameter 0)
+		(color 0 0 0 0)
 	)
 	(junction
@@
 	)
 	(no_connect
-		(at 41.91 115.57)
-	)
-	(no_connect
 		(at 80.01 64.77)
 	)
@@
 	(wire
 		(pts
+			(xy 41.91 115.57) (xy 39.37 115.57)
+		)
+		(stroke
+			(width 0)
+			(type default)
+		)
+	)
+	(wire
+		(pts
 			(xy 35.56 118.11) (xy 35.56 120.65)
 		)
@@
 	(wire
 		(pts
+			(xy 39.37 62.23) (xy 39.37 115.57)
+		)
+		(stroke
+			(width 0)
+			(type default)
+		)
+	)
+	(wire
+		(pts
 			(xy 114.3 93.98) (xy 124.46 93.98)
 		)
@@
 		)
 	)
-	(text "Need to confirm the footprint of the socket - the one included in production files \ndoes not have a model but an equivalent socket on digikey did "
+	(text "Need to confirm the footprint of the socket - the one included in production files \ndoes not have a model but an equivalent socket on digikey did so i used that downloaded model"
 		(exclude_from_sim no)
 		(at 330.454 35.814 0)
 		(effects
 			(font
+				(size 1.27 1.27)
+			)
+		)
+	)
+	(text "cw308 schematic includes note bubbles stating 'morespace' i left those out but can include if preferred"
+		(exclude_from_sim no)
+		(at 320.04 110.236 0)
+		(effects
+			(font

Commit message: updated 3 pin header to fix footprint
Parts:
- removed J1: 1x3 straight header pins, Connector_PinHeader_1.00mm:PinHeader_1x03_P1.00mm_Vertical, symbol tutorial_2_library:1x3 header 2.54mm
- added J1: 1x3 straight header pins, Connector_PinHeader_2.54mm:PinHeader_1x03_P2.54mm_Vertical, symbol tutorial_2_library:VERT_HDR_3_2.54mm
Connections:
- net GND: now also J1.1
- net at U1.12 (RF2G4_IO2): now also J1.2
- net at U1.13 (RF2G4_IO1): now also J1.3
Changed lines of the file:
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@@
-	)
-	(symbol
-		(lib_id "tutorial_2_library:1x3 header 2.54mm")
-		(at 254 90.17 0)
-		(unit 1)
-		(exclude_from_sim no)
-		(in_bom yes)
-		(on_board yes)
-		(dnp no)
-		(property "Reference" "J1"
-			(at 253.746 86.614 0)
-			(effects
-				(font
-					(size 1.27 1.27)
-				)
-				(justify left)
-			)
-		)
-		(property "Value" "1x3 straight header pins"
-			(at 265.43 161.29 0)
-			(effects
-				(font
-					(size 1.27 1.27)
-				)
-				(hide yes)
-			)
-		)
-		(property "Footprint" "Connector_PinHeader_1.00mm:PinHeader_1x03_P1.00mm_Vertical"
-			(at 254 157.48 0)
-			(effects
-				(font
-					(size 1.27 1.27)
-				)
-				(hide yes)
-			)
-		)
-		(property "Datasheet" "https://www.we-online.com/components/products/datasheet/61300311121.pdf"
-			(at 284.48 152.4 0)
-			(effects
-				(font
-					(size 1.27 1.27)
-				)
-				(hide yes)
-			)
-		)
-		(property "Description" "CONN HEADER VERT 3POS 2.54MM"
-			(at 274.32 149.86 0)
-			(effects
-				(font
-					(size 1.27 1.27)
-				)
-				(hide yes)
-			)
-		)
-		(property "Display Value" "Header"
-			(at 256.54 99.06 0)
-			(effects
-				(font
-					(size 1.27 1.27)
-				)
-				(hide yes)
-			)
-		)
-		(property "Manufacturer" "Würth Elektronik"
-			(at 245.11 161.29 0)
-			(effects
-				(font
-					(size 1.27 1.27)
-				)
-				(hide yes)
-			)
-		)
-		(property "Manufacturer Part Number" "61300311121"
-			(at 243.84 154.94 0)
-			(effects
-				(font
-					(size 1.27 1.27)
-				)
-				(hide yes)
-			)
-		)
-		(property "Supplier 1" "DigiKey"
-			(at 238.76 163.83 0)
-			(effects
-				(font
-					(size 1.27 1.27)
-				)
-				(hide yes)
-			)
-		)
-		(property "Supplier 1 Part Number" "732-5316-ND"
-			(at 266.7 163.83 0)
-			(effects
-				(font
-					(size 1.27 1.27)
-				)
-				(hide yes)
-			)
-		)
-		(property "Supplier 2" ""
-			(at 251.46 90.17 0)
-			(effects
-				(font
-					(size 1.27 1.27)
-				)
-				(hide yes)
-			)
-		)
-		(property "Supplier 2 Part Number" ""
-			(at 251.46 90.17 0)
-			(effects
-				(font
-					(size 1.27 1.27)
-				)
-				(hide yes)
-			)
-		)
-		(pin "3"
-		)
-		(pin "1"
-		)
-		(pin "2"
-		)
-		(instances
-			(project "CW312T-EFR32MG21-SOCKET"
-				(path "/ce149596-fc58-46ec-aac5-c224cd4a7fb5"
-					(reference "J1")
-					(unit 1)
-				)
-			)
-		)
 	)
 	(symbol
@@
 					(unit 1)
 				)
+			)
+		)
+	)
+	(symbol
+		(lib_id "tutorial_2_library:VERT_HDR_3_2.54mm")
+		(at 254 90.17 0)
+		(unit 1)
+		(exclude_from_sim no)
+		(in_bom yes)
+		(on_board yes)
+		(dnp no)
+		(property "Reference" "J1"
+			(at 253.746 86.614 0)
+			(effects
+				(font
+					(size 1.27 1.27)
+				)
+				(justify left)
+			)
+		)
+		(property "Value" "1x3 straight header pins"
+			(at 265.43 161.29 0)
+			(effects
+				(font
+					(size 1.27 1.27)
+				)
+				(hide yes)
+			)
+		)
+		(property "Footprint" "Connector_PinHeader_2.54mm:PinHeader_1x03_P2.54mm_Vertical"
+			(at 254 157.48 0)
+			(effects
+				(font
+					(size 1.27 1.27)
+				)
+				(hide yes)
+			)
+		)
+		(property "Datasheet" "https://www.we-online.com/components/products/datasheet/61300311121.pdf"
+			(at 284.48 152.4 0)
+			(effects
+				(font
+					(size 1.27 1.27)
+				)
+				(hide yes)
+			)
+		)
+		(property "Description" "CONN HEADER VERT 3POS 2.54MM"
+			(at 274.32 149.86 0)
+			(effects
+				(font
+					(size 1.27 1.27)
+				)
+				(hide yes)
+			)
+		)
+		(property "Display Value" "Header"
+			(at 256.54 99.06 0)
+			(effects
+				(font
+					(size 1.27 1.27)
+				)
+				(hide yes)
+			)
+		)
+		(property "Manufacturer" "Würth Elektronik"
+			(at 245.11 161.29 0)
+			(effects
+				(font
+					(size 1.27 1.27)
+				)
+				(hide yes)
+			)
+		)
+		(property "Manufacturer Part Number" "61300311121"
+			(at 243.84 154.94 0)
+			(effects
+				(font
+					(size 1.27 1.27)
+				)
+				(hide yes)
+			)
+		)
+		(property "Supplier 1" "DigiKey"
+			(at 238.76 163.83 0)
+			(effects
+				(font
+					(size 1.27 1.27)
+				)
+				(hide yes)
+			)
+		)
+		(property "Supplier 1 Part Number" "732-5316-ND"
+			(at 266.7 163.83 0)
+			(effects
+				(font
+					(size 1.27 1.27)
+				)
+				(hide yes)
+			)
+		)
+		(property "Supplier 2" ""
+			(at 251.46 90.17 0)
+			(effects
+				(font
+					(size 1.27 1.27)
+				)
+				(hide yes)
+			)
+		)
+		(property "Supplier 2 Part Number" ""
+			(at 251.46 90.17 0)
+			(effects
+				(font
+					(size 1.27 1.27)
+				)
+				(hide yes)
+			)
+		)
+		(pin "3"
+		)
+		(pin "1"
+		)
+		(pin "2"
+		)
+		(instances
+			(project ""
+				(path "/ce149596-fc58-46ec-aac5-c224cd4a7fb5"
+					(reference "J1")
+					(unit 1)
+				)

Commit message: updated schematic and pcb after library re-organization
Parts:
- removed J1: 1x3 straight header pins, Connector_PinHeader_2.54mm:PinHeader_1x03_P2.54mm_Vertical, symbol tutorial_2_library:VERT_HDR_3_2.54mm
- removed L1: IND_1K_0603, Inductor_SMD:L_0603_1608Metric, symbol tutorial_2_library:IND_1K_100MHz_0603
- removed P1: PCIEx4 EDGE CONNECTOR, tutorial_2_library:CW312_Template, symbol tutorial_2_library:CW312T-Template
- removed SJ1, SJ2, SJ3, SJ4: ~, Jumper:SolderJumper-2_P1.3mm_Bridged2Bar_Pad1.0x1.5mm, symbol tutorial_2_library:Solder_Jumper_2_NC
- removed U1: EFR32MG21A020F1024IM32-BR, tutorial_2_library:CONN_232-5205-01_3MM, symbol tutorial_2_library:EFR32MG21A020F1024IM32-BR-SOCKET
- added J1: 1x3 straight header pins, Connector_PinHeader_2.54mm:PinHeader_1x03_P2.54mm_Vertical, symbol NAE_Connectors:VERT_HDR_3_2.54mm
- added JP1, JP2, JP3, JP4: ~, Jumper:SolderJumper-2_P1.3mm_Bridged2Bar_Pad1.0x1.5mm, symbol NAE_Connectors:Solder_Jumper_2_NC
- added L1: IND_1K_0603, Inductor_SMD:L_0603_1608Metric, symbol NAE_Inductors:IND_1K_100MHz_0603
- added P1: PCIEx4 EDGE CONNECTOR, tutorial_2_library:CW312_Template, symbol NAE_Connectors:CW312T-Template
- added U1: EFR32MG21A020F1024IM32-BR, tutorial_2_library:CONN_232-5205-01_3MM, symbol NAE_Integrated_Circuits:EFR32MG21A020F1024IM32-BR-SOCKET
Connections:
- net +3V3: now also JP2.2, JP3.2, JP4.2, L1.1, P1.A26 (JTAG_VREF), P1.A5 (VCC3.3), P1.B10 (IOVREF), U1.27 (IOVDD)
- net CLKIN: now also U1.7 (HFXTAL_I)
- net FILT: now also JP1.1, P1.A3 (FILT_LP), P1.B4 (FILT_HP)
- net GND: now also J1.1, JP3.1, P1.A1 (GND), P1.A2 (GND), P1.A20 (GND), P1.A27 (GND), P1.A28 (GND), P1.A8 (GND), P1.B15 (GND), P1.B21 (GND), P1.B22 (GND), P1.B3 (GND), P1.B9 (GND), U1.10 (RFVDD), U1.11 (RFVSS), U1.33 (VSS)
- net GPIO1: now also P1.B16 (GPIO1/TX), U1.1 (PC00)
- net GPIO2: now also P1.B17 (GPIO2/RX), U1.2 (PC01)
- net GPIO3: now also P1.B18 (GPIO3), U1.3 (PC02)
- net GPIO4: now also P1.B19 (GPIO4), U1.4 (PC03)
- net RST: now also P1.A31 (JTAG_nRST), P1.B14 (nRST), U1.9 (RESETn)
- net SHUNTH: now also JP1.2, P1.B2 (SHUNTH)
- net SHUNTL: now also P1.B1 (SHUNTL), U1.24 (DECOUPLE)
- net SWCLK: now also P1.B32 (JTAG_TCK), U1.18 (PA01)
- net SWDIO: now also P1.B31 (JTAG_TMS), U1.19 (PA02)
- net TDI: now also P1.B29 (JTAG_TDI), U1.21 (PA04)
- net TDO: now also P1.B30 (JTAG_TDO), U1.20 (PA03)
- net at C8.2: now also JP2.1, U1.14 (PAVDD)
- net at C5.2: now also JP4.1, U1.25 (DVDD)
- net at C3.2: now also L1.2, U1.26 (AVDD)
- net at R2.1: now also P1.B27 (CLKOUT)
- new net: J1.2, U1.12 (RF2G4_IO2)
- new net: J1.3, U1.13 (RF2G4_IO1)
- new net: P1.B5 (FILTIN), P1.B7 (VCC1.2)
